File: SWC.kicad_sch (KiCad schematic)
At the start: 105 parts, among them J1 12V_DC_IN, J2 SWC_IN, J3 SWC_OUT, J4 USB-C 2.0 16P, J5 AUX_IN, Q3 2N7002, Q4 2N7002, Q6 2N7002, SW1 BOOT, SW2 RESET, U1 XL1509-5.0, U2 AMS1117-3.3, U3 ESP32-S3-WROOM-1-N4, U4 MCP4728, U6 TLV9004IPWR, U8 USBLC6-2SC6

Commit message: Resync C1/C2 to an Economic-eligible bulk input capacitor
C3151829 (ROQANG RVT1H101M0607) carries JLCPCB `PCBA Type: Standard Only`,
which forces the whole order onto Standard PCBA. Swap C1/C2 to C46550415
(jieerrui JVJ50V100M6x8), which is `Economic and Standard`.

Identical part class, so no layout change: 100 uF / 50 V, +/-20 %,
2000 hrs @105 C, SMD D6.3 x L7.7 mm, same `Capacitor_SMD:CP_Elec_6.3x7.7`
footprint and the same `100uF/50V` value. It also adds a published ripple
rating (140 mA @120 Hz) that the ROQANG part never listed, and widens
operation from -40..+105 C to -55..+105 C.

Schematic-only edit: the five part-identity properties (LCSC, MPN,
Manufacturer, Datasheet, Description) on each of C1 and C2. The PCB is
untouched because the footprint does not move.

This removes one of the board's two `Standard Only` parts. U3
(ESP32-S3-WROOM-1-N4, C2913197) is still `Standard Only` and still forces
Standard; every Espressif ESP32-S3-WROOM-1/-1U/-MINI-1 variant is, so that
one needs a board revision, not a substitution.

DRC and ERC are byte-for-byte unchanged from baseline (8 and 3 warnings,
0 errors, 0 unconnected).

Assisted-by: Claude Code
Parts:
- C1, C2: LCSC C3151829 -> C46550415; MPN RVT1H101M0607 -> JVJ50V100M6x8; Manufacturer ROQANG -> jieerrui
Changed lines of the file:
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@@
 			)
 		)
-		(property "Datasheet" "https://wmsc.lcsc.com/wmsc/upload/file/pdf/v2/lcsc/C3151829.pdf"
+		(property "Datasheet" "https://wmsc.lcsc.com/wmsc/upload/file/pdf/v2/lcsc/C46550415.pdf"
 			(at 52.07 34.29 0)
 			(hide yes)
@@
 			)
 		)
-		(property "Description" "100µF ±20% 50V SMD aluminium electrolytic, 6.3×7.7mm"
+		(property "Description" "100µF ±20% 50V SMD aluminium electrolytic, 6.3×7.7mm, 140mA ripple"
 			(at 52.07 34.29 0)
 			(hide yes)
@@
 			)
 		)
-		(property "Manufacturer" "ROQANG"
+		(property "Manufacturer" "jieerrui"
 			(at 52.07 34.29 0)
 			(hide yes)
@@
 			)
 		)
-		(property "MPN" "RVT1H101M0607"
+		(property "MPN" "JVJ50V100M6x8"
 			(at 52.07 34.29 0)
 			(hide yes)
@@
 			)
 		)
-		(property "LCSC" "C3151829"
+		(property "LCSC" "C46550415"
 			(at 52.07 34.29 0)
 			(hide yes)
@@
 			)
 		)
-		(property "Datasheet" "https://wmsc.lcsc.com/wmsc/upload/file/pdf/v2/lcsc/C3151829.pdf"
+		(property "Datasheet" "https://wmsc.lcsc.com/wmsc/upload/file/pdf/v2/lcsc/C46550415.pdf"
 			(at 111.76 34.29 0)
 			(hide yes)
@@
 			)
 		)
-		(property "Description" "100µF ±20% 50V SMD aluminium electrolytic, 6.3×7.7mm"
+		(property "Description" "100µF ±20% 50V SMD aluminium electrolytic, 6.3×7.7mm, 140mA ripple"
 			(at 111.76 34.29 0)
 			(hide yes)
@@
 			)
 		)
-		(property "Manufacturer" "ROQANG"
+		(property "Manufacturer" "jieerrui"
 			(at 111.76 34.29 0)
 			(hide yes)
@@
 			)
 		)
-		(property "MPN" "RVT1H101M0607"
+		(property "MPN" "JVJ50V100M6x8"
 			(at 111.76 34.29 0)
 			(hide yes)
@@
 			)
 		)
-		(property "LCSC" "C3151829"
+		(property "LCSC" "C46550415"
 			(at 111.76 34.29 0)
 			(hide yes)

Commit message: Move U3 to an Economic-eligible ESP32-S3 module (DOIT ESPS3-32-N4)
C2913197 (Espressif ESP32-S3-WROOM-1-N4) is `PCBA Type: Standard Only`, and so
is every ESP32-S3 in the WROOM-1, WROOM-1U and MINI-1 families -- all nine
WROOM-1 variants, all five WROOM-1U, all MINI-1. With C1/C2 already moved,
U3 was the only thing keeping the order on Standard.

C49164655 (DOIT ESPS3-32-N4) is `Economic and Standard` and, per its own
datasheet, a genuine clone of the WROOM-1:

  - Size 18 x 25.5 x 3 mm -- the WROOM-1 drawing, same orientation, PCB
    antenna at the module top and therefore away from the pads.
  - Pinout: all 41 pins identical by number and function, including
    IO19 = USB_D-, IO20 = USB_D+, pin 15/16 = IO3/IO46, pins 36/37 =
    RXD0/TXD0 (= IO44/IO43), pin 41 = EPAD ground.
  - Land pattern: pad 0.85 x 1.2 mm on 1.27 mm pitch, 1.5 mm pad, 2.015 mm
    edge setback, EPAD span 10.29 mm offset 7.5 mm, nine 0.9 mm EPAD vias at
    1.4/1.4/0.5 mm.

So `RF_Module:ESP32-S3-WROOM-1` is the correct footprint and the PCB is
unchanged -- schematic-only edit, six properties on U3 (Value, MPN,
Manufacturer, LCSC, Datasheet, Description).

Caveats recorded in MANUFACTURING.md rather than hidden: third-party
single source (645 stock vs 5084), DOIT's own FCC ID rather than Espressif's,
-40..+85 C (same as the WROOM-1), and no Economic-eligible PSRAM variant, so
this assumes 4 MB flash and no PSRAM. The ESP32-C3-WROOM-02 is the only other
Economic ESP32 module family and is a redesign plus firmware port.

DRC and ERC unchanged (8 and 3 warnings, 0 errors, 0 unconnected).

Assisted-by: Claude Code
Parts:
- U3: value ESP32-S3-WROOM-1-N4 -> ESPS3-32-N4; LCSC C2913197 -> C49164655; MPN ESP32-S3-WROOM-1-N4 -> ESPS3-32-N4; Manufacturer Espressif Systems -> DOIT
Changed lines of the file:
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@@
 			)
 		)
-		(property "Value" "ESP32-S3-WROOM-1-N4"
+		(property "Value" "ESPS3-32-N4"
 			(at 274.574 101.346 0)
 			(show_name no)
@@
 			)
 		)
-		(property "Datasheet" "https://wmsc.lcsc.com/wmsc/upload/file/pdf/v2/lcsc/C2913197.pdf"
+		(property "Datasheet" "https://wmsc.lcsc.com/wmsc/upload/file/pdf/v2/lcsc/C49164655.pdf"
 			(at 271.78 72.39 0)
 			(hide yes)
@@
 			)
 		)
-		(property "Description" "ESP32-S3 Wi-Fi/BLE module, 4MB flash, PCB antenna, 3.0-3.6V"
+		(property "Description" "ESP32-S3 module, 25.5×18mm 41-pin WROOM-1 form factor, 4MB flash, PCB antenna"
 			(at 271.78 72.39 0)
 			(hide yes)
@@
 			)
 		)
-		(property "Manufacturer" "Espressif Systems"
+		(property "Manufacturer" "DOIT"
 			(at 271.78 72.39 0)
 			(hide yes)
@@
 			)
 		)
-		(property "MPN" "ESP32-S3-WROOM-1-N4"
+		(property "MPN" "ESPS3-32-N4"
 			(at 271.78 72.39 0)
 			(hide yes)
@@
 			)
 		)
-		(property "LCSC" "C2913197"
+		(property "LCSC" "C49164655"
 			(at 271.78 72.39 0)
 			(hide yes)
@@
 		)
 	)
+	(symbol_instances
+		(path "/86333354-7408-43cf-8645-72f26da3f74f/bdfc9201-2ae5-4790-b433-e74bc99be33e"
+			(reference "U3")
+			(unit 1)
+			(value "ESPS3-32-N4")
+			(footprint "RF_Module:ESP32-S3-WROOM-1")
+		)
+)
 	(sheet_instances
 		(path "/"
