File: SWC.kicad_pcb (KiCad board)
At the start: 4 copper layers, 54 x 102 mm, 110 parts, among them J1 12V_DC_IN, J2 SWC_IN, J3 SWC_OUT, J4 USB-C 2.0 16P, J5 AUX_IN, Q3 2N7002, Q4 2N7002, Q6 2N7002, SW1 BOOT, SW2 RESET, U1 XL1509-5.0, U2 AMS1117-3.3, U3 ESP32-S3-WROOM-1-N4, U4 MCP4728, U6 TLV9004IPWR, U8 USBLC6-2SC6

Commit message: Update to different equivalent parts to support economical PCB assembly at JLCPCB
Parts:
- U3: value ESP32-S3-WROOM-1-N4 -> ESPS3-32-N4

Commit message: HW: bump the board to rev B; drop the JLC order marking
SWC.kicad_pcb: title-block rev A -> B. Removes the "JLCJLCJLCJLC" back-silk
string, which is a JLCPCB ordering artefact (it flags the panel so the fab
can find it) and has no place on a shipped board. One footprint's silkscreen
lines are repositioned (negative-X local coords; same geometry, tidied).

plastic_case/SWC_Enclosure.3mf: regenerated export of the enclosure.
Other:
- board text removed: "JLCJLCJLCJLC"
Changed lines of the file:
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@@
 		(title "Steering Wheel Controls Adapter")
 		(date "2026-09-10")
-		(rev "A")
+		(rev "B")
 		(company "OETSolutions, Inc.")
 	)
@@
 		(sheetname "/")
 		(sheetfile "SWC.kicad_sch")
-		(units
-			(unit
-				(name "A")
-				(pins "1" "2")
-			)
-		)
 		(attr through_hole)
 		(duplicate_pad_numbers_are_jumpers no)
 		(fp_line
-			(start 8.81126 0)
-			(end 10.81024 0)
+			(start -3 -1)
+			(end -1.00102 -1)
 			(stroke
 				(width 0.12)
@@
 		)
 		(fp_line
-			(start 9.80948 -1.00076)
-			(end 9.80948 1.00076)
+			(start -2.00178 -2.00076)
+			(end -2.00178 0.00076)
 			(stroke
 				(width 0.12)
@@
 		)
 	)
-	(gr_text "JLCJLCJLCJLC"
-		(at 50.5 71 90)
-		(layer "B.SilkS")
-		(effects
-			(font
-				(size 0.8 0.8)
-				(thickness 0.12)
-			)
-			(justify left bottom mirror)
-		)
-	)
